File: env-npd.kicad_pcb (KiCad board)
At the start: 2 copper layers, 105.4 x 99 mm, 39 parts

Commit message: Small changes, updated readme
Other:
- board text added: "https://github.com/Envious-Data/Env-NPD"
- board text removed: "Env-NPD"
Changed lines of the file:
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@@
     (mod_text_size 1 1)
     (mod_text_width 0.15)
-    (pad_size 1.5 1.5)
-    (pad_drill 0.6)
+    (pad_size 2.2 2.2)
+    (pad_drill 2.2)
     (pad_to_mask_clearance 0)
     (aux_axis_origin 0 0)
@@
       (effects (font (size 1 1) (thickness 0.15)))
     )
-    (pad 1 np_thru_hole circle (at 0 0) (size 2.2 2.2) (drill 2.2) (layers *.Cu *.Mask))
+    (pad "" np_thru_hole circle (at 0 0) (size 2.2 2.2) (drill 2.2) (layers *.Cu *.Mask Eco1.User))
   )
   (module MountingHole:MountingHole_2.2mm_M2 (layer F.Cu)
@@
       (effects (font (size 1 1) (thickness 0.15)))
     )
-    (pad 1 np_thru_hole circle (at 0 0) (size 2.2 2.2) (drill 2.2) (layers *.Cu *.Mask))
+    (pad "" np_thru_hole circle (at 0 0) (size 2.2 2.2) (drill 2.2) (layers *.Cu *.Mask Eco1.User))
   )
   (module MountingHole:MountingHole_2.2mm_M2 (layer F.Cu)
@@
       (effects (font (size 1 1) (thickness 0.15)))
     )
-    (pad 1 np_thru_hole circle (at 0 0) (size 2.2 2.2) (drill 2.2) (layers *.Cu *.Mask))
+    (pad "" np_thru_hole circle (at 0 0) (size 2.2 2.2) (drill 2.2) (layers *.Cu *.Mask Eco1.User))
   )
   (module MountingHole:MountingHole_2.2mm_M2 (layer F.Cu)
@@
       (effects (font (size 1 1) (thickness 0.15)))
     )
-    (pad 1 np_thru_hole circle (at 0 0) (size 2.2 2.2) (drill 2.2) (layers *.Cu *.Mask))
+    (pad "" np_thru_hole circle (at 0 0) (size 2.2 2.2) (drill 2.2) (layers *.Cu *.Mask Eco1.User))
   )
   (module MCU_RaspberryPi_and_Boards.pretty:RPi_Pico_SMD_TH (layer F.Cu)
@@
     (descr "Through hole straight pin header, 2x20, 2.54mm pitch, double rows")
     (tags "Through hole pin header THT 2x20 2.54mm double row")
-    (fp_text reference MCU1 (at 0 0) (layer Eco1.User)
-      (effects (font (size 1 1) (thickness 0.15)))
-    )
-    (fp_text value Pico (at 0 2.159) (layer Eco1.User)
+    (fp_text reference MCU1 (at 0 0) (layer Dwgs.User)
+      (effects (font (size 1 1) (thickness 0.15)))
+    )
+    (fp_text value Pico (at 0 2.159) (layer Dwgs.User)
       (effects (font (size 1 1) (thickness 0.15)))
     )
@@
   (gr_line (start 178.55 56.25) (end 178.55 154.45) (layer Edge.Cuts) (width 0.1))
   (gr_line (start 73.55 55.85) (end 178.15 55.85) (layer Edge.Cuts) (width 0.1))
-  (gr_text Env-NPD (at 109.35 58.35) (layer F.SilkS)
-    (effects (font (size 1.5 1.5) (thickness 0.3)))
+  (gr_text https://github.com/Envious-Data/Env-NPD (at 104.6 58.45) (layer F.SilkS)
+    (effects (font (size 1.5 1.5) (thickness 0.3)) (justify left))
   )
   (segment (start 101.4 68.95) (end 101.4 72.15) (width 0.25) (layer B.Cu) (net 1))
