File: env-npd.kicad_pcb (KiCad board)
At the start: 2 copper layers, 105.4 x 99 mm, 39 parts

Commit message: adjusted size and removed TP pads
TP pads aren't needed and they are way too close together, they may cause issues with a PCB manufacturer whos tolerances are looser than JLCPCBs
Parts:
- MCU1: footprint MCU_RaspberryPi_and_Boards.pretty:RPi_Pico_SMD_TH -> Pico:RPi_Pico_SMD_TH
- moved H1 2.55 mm to (176.0, 61.0)
- moved H3 2.55 mm to (75.8, 61.0)
Other:
- board size 105.4 x 99 mm -> 105.4 x 96 mm
